File: pcb/four_channel_audio_mixer.brd (EAGLE design)
At the start: 114 x 62 mm, 86 parts, among them J1 12V, T1 EI-14, T10 EI-14, T2 EI-14, T3 EI-14, T4 EI-14, T5 EI-14, T6 EI-14, T7 EI-14, T8 EI-14, T9 EI-14, U1 LM324D, U2 LM324D, U3 AZ1117CH-ADJTRG1, X1 SJ1-3523N, X2 SJ1-3523N, X3 SJ1-3523N, X4 SJ1-3523N, X5 SJ1-353N, X6 LED

Commit message: Version 2021-11-13
Parts:
- removed C8: 10uF, M2M-Passives:C0603
- removed C9: 100nF, M2M-Passives:C0603
- removed R1, R2: 22R, M2M-Passives:R0603
- removed R7: 100K, M2M-Passives:R0603
- removed T10, T9: EI-14, M2M-Passives:TRANSFORMER_EI14
- removed U4: (no value), M2M-IC:SOIC-14
- added R6: 100R, M2M-Passives:R0603
- added TP1: PGND, M2M-TestPoints:1X01_ROUND
- C10, C11, C12, C13, C14, C15, C16, C17: value 100pF -> 47pF
- C18, C19: value 100pF -> 0.47uF; device M2M-Passives:C0603 -> M2M-Passives:WE-4.0X5.5
- R28, R29, R30, R31, R32, R33, R34, R35: value 22K -> 10K
- R5: value 100K -> 100R
- moved R31 78.7 mm to (101.5, 14.0), turned to 90 degrees
- moved R28 70.7 mm to (99.5, 14.0), turned to 90 degrees
- moved R29 70.7 mm to (95.5, 14.0), turned to 90 degrees
- moved R30 70.7 mm to (97.5, 14.0), turned to 90 degrees
- moved R34 35.0 mm to (101.5, 17.0)
- moved R33 33.6 mm to (97.5, 17.0)
- moved R35 33.6 mm to (95.5, 17.0)
- moved C18 31.4 mm to (94.5, 44.0), turned to 270 degrees
- moved R32 31.2 mm to (99.5, 17.0)
- moved R5 26.1 mm to (94.5, 39.0), turned to 90 degrees
- moved C19 24.5 mm to (100.5, 44.0)
- moved U$1 22.4 mm to (89.5, 21.5)
- moved U$2 22.4 mm to (97.5, 33.0)
- moved C7 9.96 mm to (85.0, 29.0)
- moved R3 9.96 mm to (83.0, 29.0)
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Connections:
- removed net N$12: T9.B2, X5.3
- removed net N$19: T10.B1, T9.B1, X5.1
- removed net N$31: R2.1, U4.13, U4.14
- removed net N$33: C7.1, R3.1, R4.2, U4.10, U4.12
- net GND: now also X5.1; no longer C8.2, C9.2, U4.11
- net MIXL: now also VR5.A3; no longer C18.2, R5.1, U4.2
- net MIXR: now also VR5.B3; no longer C19.2, R7.1, U4.6
- net N$20: now also R5.1, VR5.A2; no longer T10.A1, VR5.B2
- net N$21: now also VR3.A3; no longer VR3.A1
- net N$22: now also VR3.B3; no longer VR3.B1
- net N$23: now also C19.+, R6.2; no longer T10.B2, X5.2
- net N$32: now also R6.1, VR5.B2; no longer R1.1, U4.8, U4.9
- net N$5: now also VR1.A3; no longer VR1.A1
- net N$6: now also C18.+, R5.2; no longer T9.A1, VR5.A2
- net N$7: now also VR1.B3; no longer VR1.B1
- net OUTL: now also C18.-, X5.2; no longer C18.1, R5.2, U4.1, VR5.B1
- net OUTR: now also C19.-, X5.3; no longer C19.1, R7.2, U4.7, VR5.A1
- net PGND: now also C7.1, R3.1, R4.2, TP1.1, VR1.A1, VR1.B1, VR3.A1, VR3.B1, VR5.A1, VR5.B1; no longer C8.1, R1.2, R2.2, T10.A2, T9.A2, U4.3, U4.5, VR1.A3, VR1.B3, VR3.A3, VR3.B3, VR5.A3, VR5.B3
- net VCC: no longer C9.1, U4.4
Routing:
- net N$61: track 8.15 -> 96.5 mm
- net MIXL: track 102.1 -> 16.4 mm, vias 4 -> 1
- net MIXR: track 98.6 -> 13.5 mm, vias 0 -> 1
- net N$56: track 8.65 -> 92.9 mm
- net N$59: track 18.0 -> 96.0 mm
- net N$57: track 16.7 -> 90.9 mm
- net N$66: track 27.2 -> 67.4 mm, vias 2 -> 4
- net N$69: track 15.9 -> 51.4 mm, vias 0 -> 2
- net N$62: track 13.1 -> 47.1 mm, vias 0 -> 2
- net N$19: track 32.8 -> 0.00 mm
- net N$32: track 3.59 -> 33.3 mm
- net N$65: track 17.7 -> 43.4 mm
- net N$12: track 22.8 -> 0.00 mm
- net N$7: track 35.8 -> 56.4 mm
- net OUTR: track 27.7 -> 7.53 mm
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Other:
- board text added: "2021-11-13"
- board text added: "PGND"
- board text added: "The german over engineered edition"
- board text removed: "2021-10-28"
