File: pcb/four_channel_audio_mixer.sch (EAGLE design)
At the start: 84 parts, among them J1 12V, T1 EI-14, T10 EI-14, T2 EI-14, T3 EI-14, T4 EI-14, T5 EI-14, T6 EI-14, T7 EI-14, T8 EI-14, T9 EI-14, U1 LM324D, U2 LM324D, U3 AZ1117CH-ADJTRG1, X1 SJ1-3523N, X2 SJ1-3523N, X3 SJ1-3523N, X4 SJ1-3523N, X5 SJ1-353N, X6 LED

Commit message: Version 2021-11-13
Parts:
- removed C8: 10uF, M2M-Passives:CAPC0603
- removed C9: 100nF, M2M-Passives:CAPC0603
- removed R1, R2: 22R, M2M-Passives:RESISTOR0603
- removed R7: 100K, M2M-Passives:RESISTOR0603
- removed T10, T9: EI-14, M2M-Passives:TRANSFORMEREI14
- removed U4: (no value), M2M-IC:OPAMP-LM324D
- added R6: 100R, M2M-Passives:RESISTOR0603
- added TP1: PGND, M2M-TestPoints:TESTPOINT0.1"
- C10, C11, C12, C13, C14, C15, C16, C17: value 100pF -> 47pF
- C18, C19: value 100pF -> 0.47uF; device M2M-Passives:CAPC0603 -> M2M-Passives:CAP-POL-ALUMWURTH-4.0X5.5
- R28, R29, R30, R31, R32, R33, R34, R35: value 22K -> 10K
- R5: value 100K -> 100R
Connections:
- removed net N$12: T9.B2, X5.3
- removed net N$19: T10.B1, T9.B1, X5.1
- removed net N$31: R2.1, U4G$4.IN-, U4G$4.OUT
- removed net N$33: C7.1, R3.1, R4.2, U4G$3.IN+, U4G$4.IN+
- net GND: now also X5.1; no longer C8.2, C9.2, U4G$1.VSS
- net MIXL: now also VR5L.3; no longer C18.2, R5.1, U4G$1.IN-
- net MIXR: now also VR5R.3; no longer C19.2, R7.1, U4G$2.IN-
- net N$20: now also R5.1, VR5L.2; no longer T10.A1, VR5R.2
- net N$21: now also VR3L.3; no longer VR3L.1
- net N$22: now also VR3R.3; no longer VR3R.1
- net N$23: now also C19.+, R6.2; no longer T10.B2, X5.2
- net N$32: now also R6.1, VR5R.2; no longer R1.1, U4G$3.IN-, U4G$3.OUT
- net N$5: now also VR1L.3; no longer VR1L.1
- net N$6: now also C18.+, R5.2; no longer T9.A1, VR5L.2
- net N$7: now also VR1R.3; no longer VR1R.1
- net OUTL: now also C18.-, X5.2; no longer C18.1, R5.2, U4G$1.OUT, VR5R.1
- net OUTR: now also C19.-, X5.3; no longer C19.1, R7.2, U4G$2.OUT, VR5L.1
- net PGND: now also C7.1, R3.1, R4.2, TP1.P$1, VR1L.1, VR1R.1, VR3L.1, VR3R.1, VR5L.1, VR5R.1; no longer C8.1, R1.2, R2.2, T10.A2, T9.A2, U4G$1.IN+, U4G$2.IN+, VR1L.3, VR1R.3, VR3L.3, VR3R.3, VR5L.3, VR5R.3
- net VCC: no longer C9.1, U4G$1.VCC
Other:
- moved on the sheet: R4, R5, VR1L, VR1R, VR3L, VR3R
